Commit message: Defined red material for the camera

File: ur_simulation_gz/urdf/camera.xacro (robot description, xacro)
@@ -14,4 +14,5 @@
     <xacro:property name="distortion_k2" value="0.01" />
     <xacro:property name="focal_length"  value="525" />
+    <material name="red"><color rgba="1 0 0 1"/></material>
     <joint name="${camera_name}_joint" type="fixed">
         <parent link="tool0"/>
